File: hardware/hat/sopho2sip-hat.kicad_sch (KiCad schematic)
At the start: 52 parts, among them J1 Raspberry Pi GPIO, J2 D340 Audio, J3 D340 PC-Schnittstelle, SW1 Annehmen/Auflegen, T1 600:600, T2 600:600, U1 24LC32, U2 WM8731SEDS, U3 ADuM5211, U4 AP2112K-3.3, U5 MAX3232, Y1 12.288MHz

Commit message: HAT-Schaltplan 0.2: von Hand lesbar gezeichnet (Blöcke, Leitungen, Signalfluss)
- Generator getrennt in SOLL (Verbindungen) und zeichne() (Anordnung, Leitungen, Labels zwischen Blöcken)
- Rahmen je Funktionsblock, Abblockkondensatoren an Versorgungsschienen, Trennlinien, eigene Massesymbole
- Drehung/Spiegelung und relative Textwinkel von KiCad am Testplan bestimmt
- --pruefen: ERC 0/0, KiCad-Netzliste nach Pin-Gruppen identisch mit SOLL (45 Netze)
Parts:
- JP1: value EEPROM schreiben -> WP
- SW1: value Annehmen/Auflegen -> Taste
- U5: value MAX3232 -> MAX3232E
Connections:
- net GND: now also T1.3 (SA); no longer T1.4 (SB)
- net +3V3A renamed +3.3VA
- net C1N: no longer names the net of C35.2, U5.3 (C1-)
- net C1P: no longer names the net of C35.1, U5.1 (C1+)
- net C2N: no longer names the net of C36.2, U5.5 (C2-)
- net C2P: no longer names the net of C36.1, U5.4 (C2+)
- net EEPROM_WP: no longer names the net of JP1.1 (A), R3.2, U1.7 (WP)
- net ISO_3V3 renamed +3V3_ISO
- net ISO_GND renamed GND_ISO
- net ISO_RXD: no longer names the net of U3.18 (V_{IA}), U5.12 (R1OUT)
- net ISO_TXD: no longer names the net of U3.17 (V_{OB}), U5.11 (T1IN)
- net ISO_VN: no longer names the net of C38.1, U5.6 (VS-)
- net ISO_VP: no longer names the net of C37.1, U5.2 (VS+)
- net LED1_A: no longer names the net of D1.2 (A), R6.2
- net LED2_A: no longer names the net of D2.2 (A), R7.2
- net RS232_RXD: no longer names the net of J3.2, U5.13 (R1IN)
- net RS232_TXD: no longer names the net of J3.3, U5.14 (T1OUT)
- net T1_PRI: no longer names the net of C21.2, T1.1 (AA)
- net T1_SEK: no longer names the net of C22.1
- net T1_SEK: now also T1.4 (SB); no longer T1.3 (SA)
- net T2_PRI: no longer names the net of C23.2, T2.1 (AA)
- net T2_SEK: no longer names the net of R4.1
- net T2_SEK: now also T2.4 (SB); no longer T2.3 (SA)
- net TEL_GNDA renamed GNDA
- net GNDA: now also T2.3 (SA); no longer T2.4 (SB)
- net VMID: no longer names the net of C17.1, C18.1, U2.16 (VMID)
- net XTI: no longer names the net of C10.1, U2.25 (XTI/MCLK), Y1.1
- net XTO: no longer names the net of C11.1, U2.26 (XTO), Y1.2
- net X_IN: no longer names the net of C24.2, J2.2
- net X_IN_TEILER: no longer names the net of C24.1, R4.2, R5.1
- net X_OUT: no longer names the net of C21.1, J2.1
Other:
- note added: "1200 Bd 8O1"
- note added: "1:1-Kabel zur D340,"
- note added: "2 RxD · 3 TxD · 5 GND"
- note added: "ADuM5211: Trenner mit isolierter 3,3-V-Versorgung (VSEL = GND_ISO) · dtoverlay=uart3"
- note added: "Adresse 0x50 (A0–A2 = GND); WP hoch = schreibgeschützt, JP1 schließen zum Programmieren"
- note added: "Analogversorgung 3,3 V"
- note added: "Annehmen/Auflegen (Pull-up im Pi)"
- note added: "Audio-Codec WM8731"
- note added: "Bedienung"
- note added: "D1: Telefon verbunden"
- note added: "D2: Gespräch"
- note added: "DE9-Stecker wie am PC:"
- note added: "HAT-ID-EEPROM"
- note added: "I²C 0x1A (CSB = MODE = GND) · dtoverlay=rpi-proto · Codec erzeugt die Takte (12,288 MHz)"
- note added: "LHPOUT treibt 600 Ω"
- note added: "M2,5, Raster 58 × 49 mm"
- note added: "Pi-Seite (GND)"
- note added: "RJ12 1:1 zur Audio-Buchse"
- note added: "RS-232 zur D340 (galvanisch getrennt)"
- note added: "Raspberry Pi 4 (40-polige Leiste)"
- note added: "Sprechweg zur D340 (galvanisch getrennt)"
- note added: "Telefonseite (GNDA)"
- note added: "UART3 = GPIO4/5 (PL011, kann 8O1) · I²S = GPIO18–21 · I²C1 = GPIO2/3"
- note added: "isolierte Seite (GND_ISO)"
- note added: "oben Aufnahme (X_OUT → Codec), unten Wiedergabe (Codec → X_IN); R4 = 0R, R5 unbestückt"
- note removed: "Bedienung: LEDs an GPIO23/24, Taste an GPIO25 (interner Pull-up)"
- note removed: "Codec WM8731: I²C 0x1A (CSB=0, MODE=0), Quarz 12,288 MHz,"
- note removed: "HAT-ID-EEPROM (Raspberry-Pi-HAT-Spezifikation): WP offen = schreibgeschützt, JP1 schließen zum Schreiben"
- note removed: "J3 = DE9-Stecker wie am PC: Pin 2 RxD, Pin 3 TxD, Pin 5 GND; 1:1-Kabel zur DE9-Buchse der D340 (1200 Bd 8O1)"
- note removed: "Netze per Label; erzeugt von hardware/hat/erzeuge_schaltplan.py (nicht von Hand umverdrahten)"
- note removed: "R4/R5: Teiler-Option für X_IN (Standard R4 = 0R, R5 unbestückt); Pegel per Codec einstellbar"
- note removed: "RS-232 isoliert: ADuM5211 (Digitaltrenner + isolierte 3,3 V, VSEL=GND) + MAX3232; dtoverlay=uart3 (GPIO4/5)"
- note removed: "Sopho2SIP-HAT: Raspberry Pi ⇄ ErgoLine D340 (PC-Schnittstelle RS-232, Audio-Buchse X_OUT/X_IN)"
- note removed: "Sprechweg: zwei 600:600-Übertrager trennen Telefon (TEL_GNDA) und Pi (GND) galvanisch"
- note removed: "dtoverlay=rpi-proto; LHPOUT treibt den 600-Ω-Übertrager"
