File: hardware/hat/sopho2sip-hat.kicad_sch (KiCad schematic)
At the start: 52 parts, among them J1 Raspberry Pi GPIO, J2 D340 Audio, J3 D340 PC-Schnittstelle, SW1 Taste, T1 600:600, T2 600:600, U1 24LC32, U2 WM8731SEDS, U3 ADuM5211, U4 AP2112K-3.3, U5 MAX3232E, Y1 12.288MHz

Commit message: HAT-Schaltplan: Blöcke innerhalb des Blattrahmens, Bauteiltexte neben statt über den Bauteilen
- Rahmen auf 15…405 × 15…282 mm, Sprechweg um 5,08 mm nach links (RJ12 im Rahmen)
- senkrechte R/C: Name und Wert linksbündig daneben (an Engstellen links), Abstände 10,16 mm
- JP1 senkrecht unter R3, Labels ID_SD/ID_SC frei; C33/C34/C35 entzerrt
- Prüfung unverändert: ERC 0/0, Netzliste identisch mit SOLL

Co-Authored-By: Claude Opus 5.5 <noreply@anthropic.com>
Other:
- note added: "(Pull-up im Pi)"
- note added: "Annehmen/Auflegen"
- note removed: "Annehmen/Auflegen (Pull-up im Pi)"
