File: hardware/cm4/cm4.kicad_sch (KiCad schematic)
At the start: 10 parts, among them J11 CM4 Stecker 1, J12 CM4 Stecker 2, Q10 BSS84

Commit message: CM4-Schaltplan: Einzelblock-Blätter ohne Rahmen, Inhalt zentriert
kicadgen: Steht nur ein Block auf einem Blatt, entfällt der Rahmen (sein Titel wird
Blatttitel) und der Inhalt wird auf dem Blatt zentriert (über dem Schriftfeld, auf dem
1,27-mm-Raster). Hinweistexte der CM4-Blätter an die Schaltungen gerückt.

Co-Authored-By: Claude Opus 5.5 <noreply@anthropic.com>
Other:
- note removed: "Compute Module 4"
- title: CM4 -> Compute Module 4
