File: hardware/cm4/sopho2sip-cm4.kicad_pcb (KiCad board)
At the start: 4 copper layers, 110 x 85 mm, 88 parts, among them J10 USB-C 5V/USB, J11 CM4 Stecker 1, J12 CM4 Stecker 2, J13 microSD, J14 7499010211A, J15 Lüfter 5 V, J2 D340 Audio, J3 D340 PC-Schnittstelle, Q10 BSS84, Q11 AO3400A, SW1 Taste, SW2 Konfig, SW3 Ein/Aus, T1 SM-LP-5001, T2 SM-LP-5001, U10 USBLC6-2SC6, U11 AP22804AW5, U12 TPD4E05U06DQAR, U2 TLV320AIC3204IRHBR, U3 ADuM5211, U4 AP2112K-3.3, U5 MAX3232E, U6 12MHz

Commit message: CM4-Träger: 4P4C statt DE9, CM4-Platzhalter, ausgerichtete 3D-Modelle
- Serielle Buchse J3: Würth 615004143821 (4P4C), Adapterkabel auf DE9; HAT behält DE9
- M1: CM4 als Platzhalter (Stückliste ja, Bestückungsdaten nein), offizielles STEP 1,5 mm über J11/J12
- 3D-Modelle (Würth RJ45/RJ12/RJ10, Hirose DF40, Bourns SM-LP-5001, ECS-Oszillator) als
  Modellparameter, jede Lage im Rendering geprüft; Herstellermodelle nur lokal (QUELLEN.md)
- richte_3d_aus.py: CM4-Modell laden/verschieben, Lagedatei für die Footprints
- Neu geroutet (0,127 mm Standard), DRC ohne Verstöße, 0 offene Verbindungen

Co-Authored-By: Claude Opus 5.5 <noreply@anthropic.com>
Parts:
- added M1: Raspberry Pi CM4 (z. B. CM4104032), Sopho2SIP:CM4_Modul_Platzhalter, F.Cu at (94.0, 71.0)
- J3: value D340 PC-Schnittstelle -> D340 PC (4P4C); footprint Connector_Dsub:DSUB-9_Pins_Horizontal_P2.77x2.84mm_EdgePinOffset7.70mm_Housed_MountingHolesOffset9.12mm -> Sopho2SIP:RJ10_Wuerth_615004143821_Horizontal
- moved J3 10.1 mm to (154.0, 53.9)
Connections:
- J3 pad 1: unconnected-(J3-Pad1) -> GND_ISO
Routing:
- net /CM4/USB_N: track 74.0 -> 115.4 mm, vias 0 -> 2
- net /CM4/USB_P: track 113.1 -> 73.5 mm, vias 0 -> 2
- net /Audio-Codec/I2C_SDA: track 106.5 -> 71.6 mm, vias 0 -> 2
- net /Audio-Codec/AIC_DVDD: track 25.8 -> 54.5 mm
- net Net-(U5-C2+): track 37.8 -> 10.6 mm
- net Net-(F1-Pad1): track 11.7 -> 32.0 mm
- net /Bedienung/TASTE: track 93.4 -> 74.7 mm, vias 0 -> 2
- net Net-(J10-CC1): track 32.5 -> 13.9 mm
- net /Bedienung/LED_GESPRAECH: track 78.6 -> 63.3 mm, vias 0 -> 2
- net /Bedienung/LED_TELEFON: track 76.5 -> 61.5 mm, vias 0 -> 2
- net /CM4/LED_ACT_K: track 74.8 -> 61.8 mm
- net /CM4/nRPIBOOT: track 73.1 -> 60.3 mm, vias 0 -> 1
- net /Audio-Codec/I2S_DIN: track 80.8 -> 68.2 mm, vias 0 -> 2
- net /Audio-Codec/I2S_BCLK: track 73.9 -> 86.4 mm
- net Net-(U2-IN1_R): track 7.51 -> 19.1 mm
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