File: hardware/cm4/bedienung.kicad_sch (KiCad schematic)
At the start: 14 parts, among them SW1 Taste, SW2 Konfig, SW3 Ein/Aus

Commit message: CM4-Schaltplan: Handänderungen übernommen (Handlage für 8 Blätter, 2 Texte zurückgeführt); Kastenhöhen aus gemessenen Zeichenbreiten
Other:
- moved on the sheet: D1, D2, D3, H1, H2, H3, H4, R6, R7, R8, R9, SW1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
