File: hardware/cm4/sprechweg.kicad_sch (KiCad schematic)
At the start: 9 parts, among them J2 D340 Audio, T1 600:600, T2 600:600

Commit message: CM4-Träger 0.3: Leiterplatte (4 Lagen, JLCPCB), Ein/Aus-Taster, Lüfter, lieferbare Teile
Schaltplan
- Codec TI TLV320AIC3204 statt WM8731 (abgekündigt); MCLK 12 MHz, Reset GPIO26, I²C an GPIO0/1
- Ein/Aus-Taster an GPIO3 (gpio-shutdown im Betrieb, Bootloader-Wecken im Halt)
- Lüfterblatt: AO3400A an GPIO12, Freilaufdiode, JST-PH-Anschluss; gpio-fan über SoC-Temperatur
- Konfig-Taster SW2 und Status-LED D3; Würth RJ45/RJ12, Bourns SM-LP-5001, TPD4E05U06
- reproduzierbare UUIDs (Schaltplan ↔ Platine bleiben verknüpft), eigene Footprints in hardware/bibliothek

Leiterplatte (erzeuge_layout.py)
- 110 × 85 mm, F.Cu / In1 GND / In2 +3V3 / B.Cu, JLC04161H-7628, JLCPCB-Regeln (.kicad_dru)
- CM4-Lage nach CM4IO-Referenz, Antennen-Sperrzone, isolierte Bereiche GND_ISO/GNDA mit Trennstreifen
- eigenes Fanout zu den Ebenen, Routing mit FreeRouting 1.9.0 über xvfb (2.x: Telemetrie an)
- DRC ohne Verstöße, 0 offene Verbindungen, Schaltplan ↔ Platine identisch
- Bestellliste für Digikey mit geprüftem Lagerbestand
Parts:
- J2: footprint Connector_RJ:RJ12_Amphenol_54601-x06_Horizontal -> Sopho2SIP:RJ12_Wuerth_615006138421_Horizontal
- T1, T2: value 600:600 -> SM-LP-5001; footprint (none) -> Sopho2SIP:Bourns_SM-LP-5001
Changed lines of the file:
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@@
 			(effects (font (size 1.27 1.27)))
 		)
-		(property "Footprint" "Connector_RJ:RJ12_Amphenol_54601-x06_Horizontal"
+		(property "Footprint" "Sopho2SIP:RJ12_Wuerth_615006138421_Horizontal"
 			(at 267.97 128.27 0)
 			(effects (font (size 1.27 1.27)) (hide yes))
@@
 		(instances
 			(project "sopho2sip-cm4"
-				(path "/4a9740d4-98df-4f49-9691-e6a39846794f/88d67aee-9efd-4f4b-8061-66a780267997" (reference "J2") (unit 1))
+				(path "/c325dfb5-e80f-5288-9c1c-dd309ced8908/085ac27e-fccb-53b9-9a23-a91882c9cf3e" (reference "J2") (unit 1))
 			)
 		)
@@
 			(effects (font (size 1.27 1.27)))
 		)
-		(property "Value" "600:600"
+		(property "Value" "SM-LP-5001"
 			(at 199.39 105.41 0)
 			(effects (font (size 1.27 1.27)))
 		)
-		(property "Footprint" ""
+		(property "Footprint" "Sopho2SIP:Bourns_SM-LP-5001"
 			(at 199.39 97.79 0)
 			(effects (font (size 1.27 1.27)) (hide yes))
@@
 		(instances
 			(project "sopho2sip-cm4"
-				(path "/4a9740d4-98df-4f49-9691-e6a39846794f/88d67aee-9efd-4f4b-8061-66a780267997" (reference "T1") (unit 1))
+				(path "/c325dfb5-e80f-5288-9c1c-dd309ced8908/085ac27e-fccb-53b9-9a23-a91882c9cf3e" (reference "T1") (unit 1))
 			)
 		)
@@
 			(effects (font (size 1.27 1.27)))
 		)
-		(property "Value" "600:600"
+		(property "Value" "SM-LP-5001"
 			(at 199.39 171.45 0)
 			(effects (font (size 1.27 1.27)))
 		)
-		(property "Footprint" ""
+		(property "Footprint" "Sopho2SIP:Bourns_SM-LP-5001"
 			(at 199.39 163.83 0)
 			(effects (font (size 1.27 1.27)) (hide yes))
@@
 		(instances
 			(project "sopho2sip-cm4"
-				(path "/4a9740d4-98df-4f49-9691-e6a39846794f/88d67aee-9efd-4f4b-8061-66a780267997" (reference "T2") (unit 1))
+				(path "/c325dfb5-e80f-5288-9c1c-dd309ced8908/085ac27e-fccb-53b9-9a23-a91882c9cf3e" (reference "T2") (unit 1))
 			)
 		)
@@
 		(instances
 			(project "sopho2sip-cm4"
-				(path "/4a9740d4-98df-4f49-9691-e6a39846794f/88d67aee-9efd-4f4b-8061-66a780267997" (reference "C21") (unit 1))
+				(path "/c325dfb5-e80f-5288-9c1c-dd309ced8908/085ac27e-fccb-53b9-9a23-a91882c9cf3e" (reference "C21") (unit 1))
 			)
 		)
@@
 		(instances
 			(project "sopho2sip-cm4"
-				(path "/4a9740d4-98df-4f49-9691-e6a39846794f/88d67aee-9efd-4f4b-8061-66a780267997" (reference "C22") (unit 1))
+				(path "/c325dfb5-e80f-5288-9c1c-dd309ced8908/085ac27e-fccb-53b9-9a23-a91882c9cf3e" (reference "C22") (unit 1))
 			)
 		)
@@
 		(instances
 			(project "sopho2sip-cm4"
-				(path "/4a9740d4-98df-4f49-9691-e6a39846794f/88d67aee-9efd-4f4b-8061-66a780267997" (reference "C23") (unit 1))
+				(path "/c325dfb5-e80f-5288-9c1c-dd309ced8908/085ac27e-fccb-53b9-9a23-a91882c9cf3e" (reference "C23") (unit 1))
 			)
 		)
@@
 		(instances
 			(project "sopho2sip-cm4"
-				(path "/4a9740d4-98df-4f49-9691-e6a39846794f/88d67aee-9efd-4f4b-8061-66a780267997" (reference "R4") (unit 1))
+				(path "/c325dfb5-e80f-5288-9c1c-dd309ced8908/085ac27e-fccb-53b9-9a23-a91882c9cf3e" (reference "R4") (unit 1))
 			)
 		)
@@
 		(instances
 			(project "sopho2sip-cm4"
-				(path "/4a9740d4-98df-4f49-9691-e6a39846794f/88d67aee-9efd-4f4b-8061-66a780267997" (reference "C24") (unit 1))
+				(path "/c325dfb5-e80f-5288-9c1c-dd309ced8908/085ac27e-fccb-53b9-9a23-a91882c9cf3e" (reference "C24") (unit 1))
 			)
 		)
@@
 		(instances
 			(project "sopho2sip-cm4"
-				(path "/4a9740d4-98df-4f49-9691-e6a39846794f/88d67aee-9efd-4f4b-8061-66a780267997" (reference "R5") (unit 1))
+				(path "/c325dfb5-e80f-5288-9c1c-dd309ced8908/085ac27e-fccb-53b9-9a23-a91882c9cf3e" (reference "R5") (unit 1))
 			)
 		)
@@
 		(instances
 			(project "sopho2sip-cm4"
-				(path "/4a9740d4-98df-4f49-9691-e6a39846794f/88d67aee-9efd-4f4b-8061-66a780267997" (reference "#PWRSPR001") (unit 1))
+				(path "/c325dfb5-e80f-5288-9c1c-dd309ced8908/085ac27e-fccb-53b9-9a23-a91882c9cf3e" (reference "#PWRSPR001") (unit 1))
 			)
 		)
@@
 		(instances
 			(project "sopho2sip-cm4"
-				(path "/4a9740d4-98df-4f49-9691-e6a39846794f/88d67aee-9efd-4f4b-8061-66a780267997" (reference "#PWRSPR002") (unit 1))
+				(path "/c325dfb5-e80f-5288-9c1c-dd309ced8908/085ac27e-fccb-53b9-9a23-a91882c9cf3e" (reference "#PWRSPR002") (unit 1))
 			)
 		)
@@
 		(instances
 			(project "sopho2sip-cm4"
-				(path "/4a9740d4-98df-4f49-9691-e6a39846794f/88d67aee-9efd-4f4b-8061-66a780267997" (reference "#PWRSPR003") (unit 1))
+				(path "/c325dfb5-e80f-5288-9c1c-dd309ced8908/085ac27e-fccb-53b9-9a23-a91882c9cf3e" (reference "#PWRSPR003") (unit 1))
 			)
 		)
@@
 		(instances
 			(project "sopho2sip-cm4"
-				(path "/4a9740d4-98df-4f49-9691-e6a39846794f/88d67aee-9efd-4f4b-8061-66a780267997" (reference "#PWRSPR004") (unit 1))
+				(path "/c325dfb5-e80f-5288-9c1c-dd309ced8908/085ac27e-fccb-53b9-9a23-a91882c9cf3e" (reference "#PWRSPR004") (unit 1))
 			)
 		)
@@
 		(instances
 			(project "sopho2sip-cm4"
-				(path "/4a9740d4-98df-4f49-9691-e6a39846794f/88d67aee-9efd-4f4b-8061-66a780267997" (reference "#PWRSPR005") (unit 1))
+				(path "/c325dfb5-e80f-5288-9c1c-dd309ced8908/085ac27e-fccb-53b9-9a23-a91882c9cf3e" (reference "#PWRSPR005") (unit 1))
 			)
 		)
@@
 		(instances
 			(project "sopho2sip-cm4"
-				(path "/4a9740d4-98df-4f49-9691-e6a39846794f/88d67aee-9efd-4f4b-8061-66a780267997" (reference "#PWRSPR006") (unit 1))
+				(path "/c325dfb5-e80f-5288-9c1c-dd309ced8908/085ac27e-fccb-53b9-9a23-a91882c9cf3e" (reference "#PWRSPR006") (unit 1))
 			)
 		)
@@
 		(instances
 			(project "sopho2sip-cm4"
-				(path "/4a9740d4-98df-4f49-9691-e6a39846794f/88d67aee-9efd-4f4b-8061-66a780267997" (reference "#FLGSPR001") (unit 1))
-			)
-		)
+				(path "/c325dfb5-e80f-5288-9c1c-dd309ced8908/085ac27e-fccb-53b9-9a23-a91882c9cf3e" (reference "#FLGSPR001") (unit 1))
+			)
+		)

Commit message: CM4-Schaltplan: Handänderungen übernommen (Handlage für 8 Blätter, 2 Texte zurückgeführt); Kastenhöhen aus gemessenen Zeichenbreiten
Other:
- moved on the sheet: C21
